Commit message: serial arduino commit

File: install/swerve_robot_description/share/swerve_robot_description/urdf/include/robot_parts/chassis.xacro (robot description, xacro)
@@ -1 +1 @@
-/workspaces/ros2/swerve_robot copy/src/swerve_robot_description/urdf/include/robot_parts/chassis.xacro
+/workspaces/ros2/swerve_robot/src/swerve_robot_description/urdf/include/robot_parts/chassis.xacro

File: install/swerve_robot_description/share/swerve_robot_description/urdf/include/robot_parts/steering.xacro (robot description, xacro)
@@ -1 +1 @@
-/workspaces/ros2/swerve_robot copy/src/swerve_robot_description/urdf/include/robot_parts/steering.xacro
+/workspaces/ros2/swerve_robot/src/swerve_robot_description/urdf/include/robot_parts/steering.xacro

File: install/swerve_robot_description/share/swerve_robot_description/urdf/include/robot_parts/wheel.xacro (robot description, xacro)
@@ -1 +1 @@
-/workspaces/ros2/swerve_robot copy/src/swerve_robot_description/urdf/include/robot_parts/wheel.xacro
+/workspaces/ros2/swerve_robot/src/swerve_robot_description/urdf/include/robot_parts/wheel.xacro

File: install/swerve_robot_description/share/swerve_robot_description/urdf/include/swerve_robot_base.xacro (robot description, xacro)
@@ -1 +1 @@
-/workspaces/ros2/swerve_robot copy/src/swerve_robot_description/urdf/include/swerve_robot_base.xacro
+/workspaces/ros2/swerve_robot/src/swerve_robot_description/urdf/include/swerve_robot_base.xacro

File: install/swerve_robot_description/share/swerve_robot_description/urdf/include/swerve_ros2_control.xacro (robot description, xacro)
@@ -1 +1 @@
-/workspaces/ros2/swerve_robot copy/src/swerve_robot_description/urdf/include/swerve_ros2_control.xacro
+/workspaces/ros2/swerve_robot/src/swerve_robot_description/urdf/include/swerve_ros2_control.xacro

File: install/swerve_robot_description/share/swerve_robot_description/urdf/swerve_robot.xacro (robot description, xacro)
@@ -1 +1 @@
-/workspaces/ros2/swerve_robot copy/src/swerve_robot_description/urdf/swerve_robot.xacro
+/workspaces/ros2/swerve_robot/src/swerve_robot_description/urdf/swerve_robot.xacro

File: src/swerve_robot_description/urdf/include/robot_parts/steering.xacro (robot description, xacro)
@@ -25,9 +25,9 @@
     </gazebo>
     <joint name="steering_${locationprefix}_joint" type="revolute">
-      <origin xyz="${locx} ${locy} -0.0769999999999952" rpy="0 0 0" />
+      <origin xyz="${locx} ${locy} -0.077" rpy="0 0 0" />
       <parent link="chassis_link" />
       <child link="${locationprefix}_steering_link" />
       <axis xyz="0 0 1" />
-      <limit effort="20" velocity="12.56" lower="-2.1" upper="2.1" />
+      <limit effort="20" velocity="6.28" lower="-1.57" upper="1.57" />
     </joint>
   </xacro:macro>
